Commit message: joint state-space control working

File: urdf_manipulator/urdf/urdf_manipulator.urdf (robot description, URDF)
Before this commit: robot urdf_manipulator, 6 links, 5 joints
Joints:
- joint First_joint: limit lower=-1.57 upper=1.57 effort=200 velocity=11.31 -> lower=-3.141592653589793 upper=3.141592653589793 effort=200 velocity=11.31
- joint Second_joint: limit lower=-1.57 upper=1.57 effort=200 velocity=11.31 -> lower=-3.141592653589793 upper=3.141592653589793 effort=200 velocity=11.31
- joint Third_joint: limit lower=-3.14 upper=3.14 effort=200 velocity=11.31 -> lower=-3.141592653589793 upper=3.141592653589793 effort=200 velocity=11.31
- joint base_joint: origin xyz=0.0 0.0 0.0 rpy=0 -1.57 3.14 -> xyz=0.0 0.0 0.5 rpy=0 -1.57 3.14

Commit message: complete simulation working

File: urdf_manipulator/urdf/urdf_manipulator.urdf (robot description, URDF)
Before this commit: robot urdf_manipulator, 6 links, 5 joints
Joints:
- joint base_joint: origin xyz=0.0 0.0 0.5 rpy=0 -1.57 3.14 -> xyz=0.0 0.0 0.3 rpy=0 -1.57 3.14
